Commit message: inital_pose

File: cumotion/isaac_ros_cumotion/isaac_ros_cumotion_examples/ur_config/ur.ros2_control.xacro (robot description, xacro)
@@ -1,5 +1,5 @@
 <?xml version="1.0"?>
 <robot xmlns:xacro="http://www.ros.org/wiki/xacro">
-  <xacro:macro name="ur_ros2_control" params="name initial_positions:=${dict(shoulder_pan_joint=0.0, shoulder_lift_joint=-1.57, elbow_joint=0.0, wrist_1_joint=-1.57, wrist_2_joint=0.0, wrist_3_joint=0.0)} tf_prefix">
+  <xacro:macro name="ur_ros2_control" params="name initial_positions:=${dict(shoulder_pan_joint=2.24, shoulder_lift_joint=-1.2808, elbow_joint=2.16, wrist_1_joint=-0.8848, wrist_2_joint=2.24, wrist_3_joint=0.0)} tf_prefix">
     <ros2_control name="${name}" type="system">
       <hardware>

File: ur/Universal_Robots_ROS2_Description/urdf/inc/ur_joint_control.xacro (robot description, xacro)
@@ -3,5 +3,5 @@
   <xacro:macro name="ur_joint_control_description" params="
     tf_prefix
-    initial_positions:=${dict(shoulder_pan_joint=0.0,shoulder_lift_joint=-1.57,elbow_joint=0.0,wrist_1_joint=-1.57,wrist_2_joint=0.0,wrist_3_joint=0.0)}
+    initial_positions:=${dict(shoulder_pan_joint=2.24,shoulder_lift_joint=-1.2808,elbow_joint=2.16,wrist_1_joint=-0.8848,wrist_2_joint=2.24,wrist_3_joint=0.0)}
     ">
     <joint name="${tf_prefix}shoulder_pan_joint">

File: ur/Universal_Robots_ROS2_Description/urdf/ros2_control_mock_hardware.xacro (robot description, xacro)
@@ -7,5 +7,5 @@
     tf_prefix
     mock_sensor_commands:=false
-    initial_positions:=${dict(shoulder_pan_joint=0.0,shoulder_lift_joint=-1.57,elbow_joint=0.0,wrist_1_joint=-1.57,wrist_2_joint=0.0,wrist_3_joint=0.0)}
+    initial_positions:=${dict(shoulder_pan_joint=2.24,shoulder_lift_joint=-1.2808,elbow_joint=2.16,wrist_1_joint=-0.8848,wrist_2_joint=2.24,wrist_3_joint=0.0)}
     ">
     <ros2_control name="${name}" type="system">
