Commit message: Migrate to Isaac ROS 3.2 (Humble) for AGX Orin compatibility
Switch from Isaac ROS 4.2 (Jazzy/CUDA 13.0) to Isaac ROS 3.2
(Humble/CUDA 12.6) to support AGX Orin (JetPack 6.2.x).

Changes:
- Docker: Update base image to NGC Humble tags, ROS_DISTRO=humble
- cuMotion: Replace source with release-3.2 branch
- UR Driver: Replace with humble branch (Driver, Description, Client Library)
- MoveIt Servo: Add COLCON_IGNORE (use apt ros-humble-moveit-servo)
- Servo scripts: Remove ServoCommandType (Humble API difference)
- Python: Add from __future__ import annotations for 3.10 compatibility
- Docs: Update all Jazzy/24.04 references to Humble/22.04

Co-Authored-By: Claude Opus 4.6 <noreply@anthropic.com>

File: cumotion/isaac_ros_cumotion/isaac_ros_cumotion_examples/ur_config/ur.ros2_control.xacro (robot description, xacro)
@@ -1,5 +1,5 @@
 <?xml version="1.0"?>
 <robot xmlns:xacro="http://www.ros.org/wiki/xacro">
-  <xacro:macro name="ur_ros2_control" params="name initial_positions:=${dict(shoulder_pan_joint=2.24, shoulder_lift_joint=-1.2808, elbow_joint=2.16, wrist_1_joint=-0.8848, wrist_2_joint=2.24, wrist_3_joint=0.0)} tf_prefix">
+  <xacro:macro name="ur_ros2_control" params="name initial_positions:=${dict(shoulder_pan_joint=0.0, shoulder_lift_joint=-1.57, elbow_joint=0.0, wrist_1_joint=-1.57, wrist_2_joint=0.0, wrist_3_joint=0.0)} tf_prefix">
     <ros2_control name="${name}" type="system">
       <hardware>
@@ -10,6 +10,6 @@
       <joint name="${tf_prefix}shoulder_pan_joint">
         <command_interface name="position">
-          <param name="min">-6.283185307179586</param>
-          <param name="max">6.283185307179586</param>
+          <param name="min">{-2*pi}</param>
+          <param name="max">{2*pi}</param>
         </command_interface>
         <command_interface name="velocity">
@@ -25,6 +25,6 @@
       <joint name="${tf_prefix}shoulder_lift_joint">
         <command_interface name="position">
-          <param name="min">-6.283185307179586</param>
-          <param name="max">6.283185307179586</param>
+          <param name="min">{-2*pi}</param>
+          <param name="max">{2*pi}</param>
         </command_interface>
         <command_interface name="velocity">
@@ -40,6 +40,6 @@
       <joint name="${tf_prefix}elbow_joint">
         <command_interface name="position">
-          <param name="min">-3.14159</param>
-          <param name="max">3.14159</param>
+          <param name="min">{-pi}</param>
+          <param name="max">{pi}</param>
         </command_interface>
         <command_interface name="velocity">
@@ -55,6 +55,6 @@
       <joint name="${tf_prefix}wrist_1_joint">
         <command_interface name="position">
-          <param name="min">-6.283185307179586</param>
-          <param name="max">6.283185307179586</param>
+          <param name="min">{-2*pi}</param>
+          <param name="max">{2*pi}</param>
         </command_interface>
         <command_interface name="velocity">
@@ -70,6 +70,6 @@
       <joint name="${tf_prefix}wrist_2_joint">
         <command_interface name="position">
-          <param name="min">-6.283185307179586</param>
-          <param name="max">6.283185307179586</param>
+          <param name="min">{-2*pi}</param>
+          <param name="max">{2*pi}</param>
         </command_interface>
         <command_interface name="velocity">
@@ -85,6 +85,6 @@
       <joint name="${tf_prefix}wrist_3_joint">
         <command_interface name="position">
-          <param name="min">-6.283185307179586</param>
-          <param name="max">6.283185307179586</param>
+          <param name="min">{-2*pi}</param>
+          <param name="max">{2*pi}</param>
         </command_interface>
         <command_interface name="velocity">

File: cumotion/isaac_ros_cumotion/isaac_ros_cumotion_examples/ur_config/ur.urdf.xacro (robot description, xacro)
@@ -1,48 +1,13 @@
 <?xml version="1.0"?>
-<robot xmlns:xacro="http://wiki.ros.org/xacro" name="ur">
-   <!-- robot name parameter -->
-   <xacro:arg name="name" default="ur"/>
-   <xacro:arg name="initial_positions_file" default="$(find isaac_ros_cumotion_examples)/ur_config/initial_positions.yaml"/>
-  <xacro:property name="initial_positions_file" value="$(arg initial_positions_file)"/>
-   <!-- import main macro -->
-   <xacro:include filename="$(find ur_description)/urdf/ur_macro.xacro"/>
-   <!-- import ros2_control description -->
-   <xacro:include filename="ur.ros2_control.xacro" />
-   <!-- possible 'ur_type' values: ur3, ur3e, ur5, ur5e, ur10, ur10e, ur16e, ur20, ur30 -->
-   <!-- the default value should raise an error in case this was called without defining the type -->
-   <xacro:arg name="ur_type" default="ur5x"/>
-   <!-- parameters -->
-   <xacro:arg name="tf_prefix" default="" />
-   <xacro:arg name="joint_limit_params" default="$(find ur_description)/config/$(arg ur_type)/joint_limits.yaml"/>
-   <xacro:arg name="kinematics_params" default="$(find ur_description)/config/$(arg ur_type)/default_kinematics.yaml"/>
-   <xacro:arg name="physical_params" default="$(find ur_description)/config/$(arg ur_type)/physical_parameters.yaml"/>
-   <xacro:arg name="visual_params" default="$(find ur_description)/config/$(arg ur_type)/visual_parameters.yaml"/>
-   <xacro:arg name="transmission_hw_interface" default=""/>
-   <xacro:arg name="safety_limits" default="false"/>
-   <xacro:arg name="safety_pos_margin" default="0.15"/>
-   <xacro:arg name="safety_k_position" default="20"/>
-   <xacro:arg name="force_abs_paths" default="false"/>
-   <!-- create link fixed to the "world" -->
-   <link name="world" />
-   <!-- arm -->
-   <xacro:ur_robot
-     name="$(arg name)"
-     tf_prefix="$(arg tf_prefix)"
-     parent="world"
-     joint_limits_parameters_file="$(arg joint_limit_params)"
-     kinematics_parameters_file="$(arg kinematics_params)"
-     physical_parameters_file="$(arg physical_params)"
-     visual_parameters_file="$(arg visual_params)"
-     safety_limits="$(arg safety_limits)"
-     safety_pos_margin="$(arg safety_pos_margin)"
-     safety_k_position="$(arg safety_k_position)"
-     force_abs_paths="$(arg force_abs_paths)"
-     >
-     <origin xyz="0 0 0" rpy="0 0 0" />          <!-- position robot in the world -->
-   </xacro:ur_robot>
-  <!-- ros2_control -->
-  <xacro:ur_ros2_control
-    name="UR_IsaacSim"
-    tf_prefix="$(arg tf_prefix)"
-    initial_positions="${xacro.load_yaml(initial_positions_file)}"/>
+<robot xmlns:xacro="http://www.ros.org/wiki/xacro" name="$(arg ur_type)">
+    <xacro:arg name="ur_type" default="ur"/>
+    <xacro:arg name="use_fake_hardware" default="true" />
+    <xacro:arg name="name" default="ur10e" />
+    <!-- Do not add ROS2 control from default UR package, add TopicBasedROS2 Control -->
+    <xacro:arg name="generate_ros2_control_tag" default="false" />
+    <!-- Import UR URDF file -->
+    <xacro:include filename="$(find isaac_ros_cumotion_examples)/ur_config/ur_sim.urdf.xacro" />
+    <!-- Import UR ros2_control description -->
+    <xacro:include filename="ur.ros2_control.xacro" />
+    <xacro:ur_ros2_control name="URFakeSystem" tf_prefix="" />
 </robot>

File: cumotion/isaac_ros_cumotion/isaac_ros_cumotion_robot_description/urdf/ur10e_robotiq_2f_140.urdf (robot description, URDF)
Before this commit: robot ur10e_robot, 25 links, 24 joints
Links:
- removed link insertion_frame
Joints:
- removed joint insertion_joint

File: cumotion/isaac_ros_cumotion/isaac_ros_cumotion_robot_description/urdf/ur5e_robotiq_2f_140.urdf (robot description, URDF)
Before this commit: robot ur5e_robot, 25 links, 24 joints
Links:
- removed link insertion_frame
Joints:
- removed joint insertion_joint

File: cumotion/isaac_ros_cumotion/isaac_ros_cumotion_robot_description/urdf/ur5e_robotiq_2f_85.urdf (robot description, URDF)
Before this commit: robot robotiq_gripper, 25 links, 24 joints
Links:
- removed link insertion_frame
Joints:
- removed joint insertion_joint
